File: prj 3 - mcu datalogger.kicad_sch (KiCad schematic)
At the start: 25 parts, among them U1 DS1337S+, U2 24LC1025, U3 24LC1025, U4 ATMEGA328P-AU, Y1 33.768 KHz, Y2 16MHz

Commit message: allocated GND and VCC nets to the power net class
Connections:
- net VCC: now also R6.1
Other:
- sheet connectors ports: added D2, D3, D4, D5, D6, D7, D8, GND, MISO, MOSI, RESET, RX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; removed none
